Commit message: Update circular robot model

File: urdf/robot_circular.xacro (robot description, xacro)
@@ -22,5 +22,5 @@
       <origin xyz="0 0 0.05" rpy=" 0 0 0"/>
       <geometry>
-        <cylinder length="0.15" radius="0.3"/>
+        <cylinder length="0.1" radius="0.2"/>
       </geometry>
     </collision>
@@ -28,29 +28,53 @@
       <origin xyz="0 0 0.05" rpy=" 0 0 0"/>
       <geometry>
-        <cylinder length="0.15" radius="0.3"/>
-      </geometry>
-    </visual>
-    <collision name='back_caster_collision'>
-      <origin xyz="-0.125 0 -0.0375" rpy=" 0 0 0"/>
-      <geometry>
-        <sphere radius="0.0375"/>
-      </geometry>
-    </collision>
-    <visual name='back_caster_visual'>
-      <origin xyz="-0.125 0 -0.0375" rpy=" 0 0 0"/>
-      <geometry>
-        <sphere radius="0.0375"/>
-      </geometry>
-    </visual>
-    <collision name='front_caster_collision'>
-      <origin xyz="0.125 0 -0.0375" rpy=" 0 0 0"/>
-      <geometry>
-        <sphere radius="0.0375"/>
-      </geometry>
-    </collision>
-    <visual name='front_caster_visual'>
-      <origin xyz="0.125 0 -0.0375" rpy=" 0 0 0"/>
-      <geometry>
-        <sphere radius="0.0375"/>
+        <cylinder length="0.1" radius="0.2"/>
+      </geometry>
+    </visual>
+    <collision name='right_up_caster_collision'>
+      <origin xyz="-0.1 0.1 -0.0" rpy=" 0 0 0"/>
+      <geometry>
+        <sphere radius="0.05"/>
+      </geometry>
+    </collision>
+    <visual name='right_up_caster_visual'>
+      <origin xyz="-0.1 0.1 -0.0" rpy=" 0 0 0"/>
+      <geometry>
+        <sphere radius="0.05"/>
+      </geometry>
+    </visual>
+    <collision name='right_down_caster_collision'>
+      <origin xyz="0.1 0.1 -0.0" rpy=" 0 0 0"/>
+      <geometry>
+        <sphere radius="0.05"/>
+      </geometry>
+    </collision>
+    <visual name='right_down_caster_visual'>
+      <origin xyz="0.1 0.1 -0.0" rpy=" 0 0 0"/>
+      <geometry>
+        <sphere radius="0.05"/>
+      </geometry>
+    </visual>
+    <collision name='left_up_caster_collision'>
+      <origin xyz="-0.1 -0.1 -0.0" rpy=" 0 0 0"/>
+      <geometry>
+        <sphere radius="0.05"/>
+      </geometry>
+    </collision>
+    <visual name='left_up_caster_visual'>
+      <origin xyz="-0.1 -0.1 -0.0" rpy=" 0 0 0"/>
+      <geometry>
+        <sphere radius="0.05"/>
+      </geometry>
+    </visual>
+    <collision name='left_down_caster_collision'>
+      <origin xyz="0.1 -0.1 -0.0" rpy=" 0 0 0"/>
+      <geometry>
+        <sphere radius="0.05"/>
+      </geometry>
+    </collision>
+    <visual name='left_down_caster_visual'>
+      <origin xyz="0.1 -0.1 -0.0" rpy=" 0 0 0"/>
+      <geometry>
+        <sphere radius="0.05"/>
       </geometry>
     </visual>
@@ -69,5 +93,5 @@
       <origin xyz="0 0 0" rpy=" 0 1.5707 1.5707"/>
       <geometry>
-        <cylinder radius="0.075" length="0.05"/>
+        <cylinder radius="0.05" length="0.05"/>
       </geometry>
     </collision>
@@ -75,5 +99,5 @@
       <origin xyz="0 0 0" rpy=" 0 1.5707 1.5707"/>
       <geometry>
-        <cylinder radius="0.075" length="0.05"/>
+        <cylinder radius="0.05" length="0.05"/>
       </geometry>
     </visual>
@@ -92,5 +116,5 @@
       <origin xyz="0 0 0" rpy=" 0 1.5707 1.5707"/>
       <geometry>
-        <cylinder radius="0.075" length="0.05"/>
+        <cylinder radius="0.05" length="0.05"/>
       </geometry>
     </collision>
@@ -98,10 +122,10 @@
       <origin xyz="0 0 0" rpy=" 0 1.5707 1.5707"/>
       <geometry>
-        <cylinder radius="0.075" length="0.05"/>
+        <cylinder radius="0.05" length="0.05"/>
       </geometry>
     </visual>
   </link>
   <joint type="continuous" name="left_wheel_hinge">
-    <origin xyz="0 0.2 0" rpy="0 0 0"/>
+    <origin xyz="0 0.15 0" rpy="0 0 0"/>
     <child link="left_wheel"/>
     <parent link="chassis"/>
@@ -111,5 +135,5 @@
   </joint>
   <joint type="continuous" name="right_wheel_hinge">
-    <origin xyz="0 -0.2 0" rpy="0 0 0"/>
+    <origin xyz="0 -0.15 0" rpy="0 0 0"/>
     <child link="right_wheel"/>
     <parent link="chassis"/>
@@ -142,5 +166,5 @@
   </link>
   <joint type="fixed" name="camera_joint">
-    <origin xyz="0.3 0 0.075" rpy="0 0 0"/>
+    <origin xyz="0.2 0 0.05" rpy="0 0 0"/>
     <child link="camera"/>
     <parent link="chassis"/>
@@ -170,5 +194,5 @@
   </link>
   <joint type="fixed" name="hokuyo_joint">
-    <origin xyz="0.0 0 0.15" rpy="0 0 0"/>
+    <origin xyz="0.0 0 0.1" rpy="0 0 0"/>
     <child link="hokuyo"/>
     <parent link="chassis"/>

Commit message: Update robot circular model

File: urdf/robot_circular.xacro (robot description, xacro)
@@ -1,5 +1,5 @@
 <?xml version='1.0'?>
-<robot name="robot_circular" xmlns:xacro="http://www.ros.org/wiki/xacro">
-  <xacro:include filename="$(find udacity_bot)/urdf/robot_circular.gazebo" />
+<robot name="udacity_bot" xmlns:xacro="http://www.ros.org/wiki/xacro">
+  <xacro:include filename="$(find udacity_bot)/urdf/udacity_bot.gazebo" />
   <link name="robot_footprint"></link>
   <joint name="robot_footprint_joint" type="fixed">
@@ -11,6 +11,6 @@
     <pose>0 0 0.1 0 0 0</pose>
     <inertial>
-      <mass value="1.5"/>
-      <origin xyz="0.0 0 0.05" rpy=" 0 0 0"/>
+      <mass value="15.0"/>
+      <origin xyz="0.0 0 0" rpy=" 0 0 0"/>
       <inertia
           ixx="0.1" ixy="0" ixz="0"
@@ -20,59 +20,35 @@
     </inertial>
     <collision name='collision'>
-      <origin xyz="0 0 0.05" rpy=" 0 0 0"/>
+      <origin xyz="0 0 0" rpy=" 0 0 0"/>
       <geometry>
-        <cylinder length="0.1" radius="0.2"/>
+        <cylinder length="0.1" radius="0.25"/>
       </geometry>
     </collision>
     <visual name='chassis_visual'>
-      <origin xyz="0 0 0.05" rpy=" 0 0 0"/>
+      <origin xyz="0 0 0" rpy=" 0 0 0"/>
       <geometry>
-        <cylinder length="0.1" radius="0.2"/>
+        <cylinder length="0.1" radius="0.25"/>
       </geometry>
     </visual>
-    <collision name='right_up_caster_collision'>
-      <origin xyz="-0.1 0.1 -0.0" rpy=" 0 0 0"/>
+    <collision name='back_caster_collision'>
+      <origin xyz="-0.15 0 -0.05" rpy=" 0 0 0"/>
       <geometry>
-        <sphere radius="0.05"/>
+        <sphere radius="0.0499"/>
       </geometry>
     </collision>
-    <visual name='right_up_caster_visual'>
-      <origin xyz="-0.1 0.1 -0.0" rpy=" 0 0 0"/>
+    <visual name='back_caster_visual'>
+      <origin xyz="-0.15 0 -0.05" rpy=" 0 0 0"/>
       <geometry>
         <sphere radius="0.05"/>
       </geometry>
     </visual>
-    <collision name='right_down_caster_collision'>
-      <origin xyz="0.1 0.1 -0.0" rpy=" 0 0 0"/>
+    <collision name='front_caster_collision'>
+      <origin xyz="0.15 0 -0.05" rpy=" 0 0 0"/>
       <geometry>
-        <sphere radius="0.05"/>
+        <sphere radius="0.0499"/>
       </geometry>
     </collision>
-    <visual name='right_down_caster_visual'>
-      <origin xyz="0.1 0.1 -0.0" rpy=" 0 0 0"/>
-      <geometry>
-        <sphere radius="0.05"/>
-      </geometry>
-    </visual>
-    <collision name='left_up_caster_collision'>
-      <origin xyz="-0.1 -0.1 -0.0" rpy=" 0 0 0"/>
-      <geometry>
-        <sphere radius="0.05"/>
-      </geometry>
-    </collision>
-    <visual name='left_up_caster_visual'>
-      <origin xyz="-0.1 -0.1 -0.0" rpy=" 0 0 0"/>
-      <geometry>
-        <sphere radius="0.05"/>
-      </geometry>
-    </visual>
-    <collision name='left_down_caster_collision'>
-      <origin xyz="0.1 -0.1 -0.0" rpy=" 0 0 0"/>
-      <geometry>
-        <sphere radius="0.05"/>
-      </geometry>
-    </collision>
-    <visual name='left_down_caster_visual'>
-      <origin xyz="0.1 -0.1 -0.0" rpy=" 0 0 0"/>
+    <visual name='front_caster_visual'>
+      <origin xyz="0.15 0 -0.05" rpy=" 0 0 0"/>
       <geometry>
         <sphere radius="0.05"/>
@@ -82,5 +58,5 @@
   <link name='left_wheel'>
     <inertial>
-      <mass value="0.4"/>
+      <mass value="2.5"/>
       <origin xyz="0.0 0 0" rpy=" 0 1.5707 1.5707"/>
       <inertia
@@ -105,5 +81,5 @@
   <link name='right_wheel'>
     <inertial>
-      <mass value="0.4"/>
+      <mass value="2.5"/>
       <origin xyz="0.0 0 0" rpy=" 0 1.5707 1.5707"/>
       <inertia
@@ -127,5 +103,5 @@
   </link>
   <joint type="continuous" name="left_wheel_hinge">
-    <origin xyz="0 0.15 0" rpy="0 0 0"/>
+    <origin xyz="0 0.28 -0.05" rpy="0 0 0"/>
     <child link="left_wheel"/>
     <parent link="chassis"/>
@@ -135,5 +111,5 @@
   </joint>
   <joint type="continuous" name="right_wheel_hinge">
-    <origin xyz="0 -0.15 0" rpy="0 0 0"/>
+    <origin xyz="0 -0.28 -0.05" rpy="0 0 0"/>
     <child link="right_wheel"/>
     <parent link="chassis"/>
@@ -166,5 +142,5 @@
   </link>
   <joint type="fixed" name="camera_joint">
-    <origin xyz="0.2 0 0.05" rpy="0 0 0"/>
+    <origin xyz="0.3 0 0.0" rpy="0 0 0"/>
     <child link="camera"/>
     <parent link="chassis"/>
