Commit message: Update circular base robot

File: urdf/robot_circular_bkp.xacro (robot description, xacro)
@@ -11,6 +11,6 @@
     <pose>0 0 0.1 0 0 0</pose>
     <inertial>
-      <mass value="8.0"/>
-      <origin xyz="0.0 0 0.04" rpy=" 0 0 0"/>
+      <mass value="1.5"/>
+      <origin xyz="0.0 0 0.08" rpy=" 0 0 0"/>
       <inertia
           ixx="0.1" ixy="0" ixz="0"
@@ -20,66 +20,44 @@
     </inertial>
     <collision name='collision'>
-      <origin xyz="0 0 0.04" rpy=" 0 0 0"/>
+      <origin xyz="0 0 0.08" rpy=" 0 0 0"/>
       <geometry>
-        <cylinder length="0.12" radius="0.25"/>
+        <cylinder length="0.1" radius="0.2"/>
       </geometry>
     </collision>
     <visual name='chassis_visual'>
-      <origin xyz="0 0 0.04" rpy=" 0 0 0"/>
+      <origin xyz="0 0 0.08" rpy=" 0 0 0"/>
       <geometry>
-        <cylinder length="0.12" radius="0.25"/>
+        <cylinder length="0.1" radius="0.2"/>
       </geometry>
     </visual>
     <collision name='back_caster_collision'>
-      <origin xyz="-0.15 0 -0.05" rpy=" 0 0 0"/>
+      <origin xyz="-0.15 0 0.0" rpy=" 0 0 0"/>
       <geometry>
-        <sphere radius="0.0499"/>
+        <sphere radius="0.03"/>
       </geometry>
     </collision>
     <visual name='back_caster_visual'>
-      <origin xyz="-0.15 0 -0.05" rpy=" 0 0 0"/>
+      <origin xyz="-0.15 0 0.0" rpy=" 0 0 0"/>
       <geometry>
-        <sphere radius="0.05"/>
+        <sphere radius="0.03"/>
       </geometry>
     </visual>
     <collision name='front_caster_collision'>
-      <origin xyz="0.15 0 -0.05" rpy=" 0 0 0"/>
+      <origin xyz="0.15 0 0.0" rpy=" 0 0 0"/>
       <geometry>
-        <sphere radius="0.0499"/>
+        <sphere radius="0.03"/>
       </geometry>
     </collision>
     <visual name='front_caster_visual'>
-      <origin xyz="0.15 0 -0.05" rpy=" 0 0 0"/>
+      <origin xyz="0.15 0 0.0" rpy=" 0 0 0"/>
       <geometry>
-        <sphere radius="0.05"/>
+        <sphere radius="0.03"/>
       </geometry>
     </visual>
   </link>
-  <link name='rectangle_link'>
-    <inertial>
-      <mass value="4.0"/>
-      <origin xyz="0.0 0 0.0" rpy=" 0 1.57075 0"/>
-      <inertia
-          ixx="0.1" ixy="0" ixz="0"
-          iyy="0.1" iyz="0"
-          izz="0.1"
-      />
-    </inertial>
-   <visual>
-    <origin xyz="0.0 0 0.0" rpy=" 0 1.57075  0"/>
-    <geometry>
-     <box size="0.3 0.12 0.06"/>
-    </geometry>
-   </visual>
-  </link>
-  <joint name='base_to_rectangle_link' type="fixed">
-   <parent link="chassis"/>
-   <child link="rectangle_link"/>
-   <origin xyz="0.15 0.0 0.25"/>
-  </joint>
   <link name='left_wheel'>
     <inertial>
-      <mass value="2.5"/>
-      <origin xyz="0.0 0 0.05" rpy=" 0 1.5707 1.5707"/>
+      <mass value="0.4"/>
+      <origin xyz="0.0 0 0" rpy=" 0 1.5707 1.5707"/>
       <inertia
           ixx="0.1" ixy="0" ixz="0"
@@ -89,13 +67,13 @@
     </inertial>
     <collision name='collision'>
-      <origin xyz="0 0 0.05" rpy=" 0 1.5707 1.5707"/>
+      <origin xyz="0 0 0" rpy=" 0 1.5707 1.5707"/>
       <geometry>
-        <cylinder radius="0.1" length="0.05"/>
+        <cylinder radius="0.03" length="0.03"/>
       </geometry>
     </collision>
     <visual name='left_wheel_visual'>
-      <origin xyz="0 0 0.05" rpy=" 0 1.5707 1.5707"/>
+      <origin xyz="0 0 0" rpy=" 0 1.5707 1.5707"/>
       <geometry>
-        <cylinder radius="0.1" length="0.05"/>
+        <cylinder radius="0.03" length="0.03"/>
       </geometry>
     </visual>
@@ -103,6 +81,6 @@
   <link name='right_wheel'>
     <inertial>
-      <mass value="2.5"/>
-      <origin xyz="0.0 0 0.05" rpy=" 0 1.5707 1.5707"/>
+      <mass value="0.4"/>
+      <origin xyz="0.0 0 0" rpy=" 0 1.5707 1.5707"/>
       <inertia
           ixx="0.1" ixy="0" ixz="0"
@@ -112,18 +90,18 @@
     </inertial>
     <collision name='collision'>
-      <origin xyz="0 0 0.05" rpy=" 0 1.5707 1.5707"/>
+      <origin xyz="0 0 0" rpy=" 0 1.5707 1.5707"/>
       <geometry>
-        <cylinder radius="0.1" length="0.05"/>
+        <cylinder radius="0.03" length="0.03"/>
       </geometry>
     </collision>
     <visual name='right_wheel_visual'>
-      <origin xyz="0 0 0.05" rpy=" 0 1.5707 1.5707"/>
+      <origin xyz="0 0 0" rpy=" 0 1.5707 1.5707"/>
       <geometry>
-        <cylinder radius="0.1" length="0.05"/>
+        <cylinder radius="0.03" length="0.03"/>
       </geometry>
     </visual>
   </link>
   <joint type="continuous" name="left_wheel_hinge">
-    <origin xyz="0 0.28 -0.05" rpy="0 0 0"/>
+    <origin xyz="0 0.15 0" rpy="0 0 0"/>
     <child link="left_wheel"/>
     <parent link="chassis"/>
@@ -133,5 +111,5 @@
   </joint>
   <joint type="continuous" name="right_wheel_hinge">
-    <origin xyz="0 -0.28 -0.05" rpy="0 0 0"/>
+    <origin xyz="0 -0.15 0" rpy="0 0 0"/>
     <child link="right_wheel"/>
     <parent link="chassis"/>
@@ -164,5 +142,5 @@
   </link>
   <joint type="fixed" name="camera_joint">
-    <origin xyz="0.3 0.0 0.075" rpy="0 0 0"/>
+    <origin xyz="0.2 0 0.1" rpy="0 0 0"/>
     <child link="camera"/>
     <parent link="chassis"/>
@@ -192,5 +170,5 @@
   </link>
   <joint type="fixed" name="hokuyo_joint">
-    <origin xyz="0.15 0 0.425" rpy="0 0 0"/>
+    <origin xyz="0.0 0 0.2" rpy="0 0 0"/>
     <child link="hokuyo"/>
     <parent link="chassis"/>
