Commit message: Final changes to custom robot and model parameters
- Update AMCL parameters to localize Udacity as well as Custom Slim Robot
- Add ReadMe

File: urdf/robot_custom.xacro (robot description, xacro)
@@ -22,5 +22,5 @@
       <origin xyz="0 0 0" rpy=" 0 0 0"/>
       <geometry>
-        <box size=".2 .3 .08"/>
+        <box size=".25 .12 .04"/>
       </geometry>
     </collision>
@@ -28,29 +28,29 @@
       <origin xyz="0 0 0" rpy=" 0 0 0"/>
       <geometry>
-        <box size=".2 .3 .08"/>
+        <box size=".25 .12 .04"/>
       </geometry>
     </visual>
     <collision name='back_caster_collision'>
-      <origin xyz="-0.05 0 -0.05" rpy=" 0 0 0"/>
-      <geometry>
-        <sphere radius="0.0499"/>
+      <origin xyz="-0.09 0 -0.025" rpy=" 0 0 0"/>
+      <geometry>
+        <sphere radius="0.02499"/>
       </geometry>
     </collision>
     <visual name='back_caster_visual'>
-      <origin xyz="-0.05 0  -0.05" rpy=" 0 0 0"/>
-      <geometry>
-        <sphere radius="0.05"/>
+      <origin xyz="-0.09 0  -0.025" rpy=" 0 0 0"/>
+      <geometry>
+        <sphere radius="0.025"/>
       </geometry>
     </visual>
     <collision name='front_caster_collision'>
-      <origin xyz="0.05 0 -0.05" rpy=" 0 0 0"/>
-      <geometry>
-        <sphere radius="0.0499"/>
+      <origin xyz="0.09 0 -0.025" rpy=" 0 0 0"/>
+      <geometry>
+        <sphere radius="0.02499"/>
       </geometry>
     </collision>
     <visual name='front_caster_visual'>
-      <origin xyz="0.05 0 -0.05" rpy=" 0 0 0"/>
-      <geometry>
-        <sphere radius="0.05"/>
+      <origin xyz="0.09 0 -0.025" rpy=" 0 0 0"/>
+      <geometry>
+        <sphere radius="0.025"/>
       </geometry>
     </visual>
@@ -58,5 +58,5 @@
     <link name='rectangle_link'>
     <inertial>
-      <mass value="5.0"/>
+      <mass value="2.0"/>
       <origin xyz="0.0 0 0.0" rpy=" 0 1.57075 0"/>
       <inertia
@@ -80,5 +80,5 @@
   <link name='cylindrical_link'>
     <inertial>
-      <mass value="3.0"/>
+      <mass value="4.0"/>
       <origin xyz="0.0 0 0.0" rpy=" 0 0 0"/>
       <inertia
@@ -102,22 +102,22 @@
   <link name='left_wheel'>
     <inertial>
-      <mass value="2.5"/>
-      <origin xyz="0.0 0 0.05" rpy=" 0 1.5707 1.5707"/>
-      <inertia
-          ixx="0.1" ixy="0" ixz="0"
-          iyy="0.1" iyz="0"
-          izz="0.1"
-      />
-    </inertial>
-    <collision name='collision'>
-      <origin xyz="0 0 0.05" rpy=" 0 1.5707 1.5707"/>
-      <geometry>
-        <cylinder radius="0.05" length="0.05"/>
+      <mass value="0.5"/>
+      <origin xyz="0.0 0 0" rpy=" 0 1.5707 1.5707"/>
+      <inertia
+          ixx="0.1" ixy="0" ixz="0"
+          iyy="0.1" iyz="0"
+          izz="0.1"
+      />
+    </inertial>
+    <collision name='collision'>
+      <origin xyz="0 0 0" rpy=" 0 1.5707 1.5707"/>
+      <geometry>
+        <cylinder radius="0.05" length="0.025"/>
       </geometry>
     </collision>
     <visual name='left_wheel_visual'>
-      <origin xyz="0 0 0.05" rpy=" 0 1.5707 1.5707"/>
-      <geometry>
-        <cylinder radius="0.05" length="0.05"/>
+      <origin xyz="0 0 0" rpy=" 0 1.5707 1.5707"/>
+      <geometry>
+        <cylinder radius="0.05" length="0.025"/>
       </geometry>
     </visual>
@@ -125,39 +125,39 @@
   <link name='right_wheel'>
     <inertial>
-      <mass value="2.5"/>
-      <origin xyz="0.0 0 0.05" rpy=" 0 1.5707 1.5707"/>
-      <inertia
-          ixx="0.1" ixy="0" ixz="0"
-          iyy="0.1" iyz="0"
-          izz="0.1"
-      />
-    </inertial>
-    <collision name='collision'>
-      <origin xyz="0 0 0.05" rpy=" 0 1.5707 1.5707"/>
-      <geometry>
-        <cylinder radius="0.05" length="0.05"/>
+      <mass value="0.5"/>
+      <origin xyz="0.0 0 -0.05" rpy=" 0 1.5707 1.5707"/>
+      <inertia
+          ixx="0.1" ixy="0" ixz="0"
+          iyy="0.1" iyz="0"
+          izz="0.1"
+      />
+    </inertial>
+    <collision name='collision'>
+      <origin xyz="0 0 0" rpy=" 0 1.5707 1.5707"/>
+      <geometry>
+        <cylinder radius="0.05" length="0.025"/>
       </geometry>
     </collision>
     <visual name='right_wheel_visual'>
-      <origin xyz="0 0 0.05" rpy=" 0 1.5707 1.5707"/>
-      <geometry>
-        <cylinder radius="0.05" length="0.05"/>
+      <origin xyz="0 0 0" rpy=" 0 1.5707 1.5707"/>
+      <geometry>
+        <cylinder radius="0.05" length="0.025"/>
       </geometry>
     </visual>
   </link>
   <joint type="continuous" name="left_wheel_hinge">
-    <origin xyz="0 0.18 -0.1" rpy="0 0 0"/>
+    <origin xyz="0 0.1 0.0" rpy="0 0 0"/>
     <child link="left_wheel"/>
     <parent link="chassis"/>
     <axis xyz="0 1 0" rpy="0 0 0"/>
-    <limit effort="10000" velocity="1000"/>
+    <limit effort="5000" velocity="500"/>
     <dynamics damping="1.0" friction="1.0"/>
   </joint>
   <joint type="continuous" name="right_wheel_hinge">
-    <origin xyz="0 -0.18 -0.1" rpy="0 0 0"/>
+    <origin xyz="0 -0.1 0.0" rpy="0 0 0"/>
     <child link="right_wheel"/>
     <parent link="chassis"/>
     <axis xyz="0 1 0" rpy="0 0 0"/>
-    <limit effort="10000" velocity="1000"/>
+    <limit effort="5000" velocity="500"/>
     <dynamics damping="1.0" friction="1.0"/>
   </joint>
